File: EAGLE/Tiny Tetris v1.3.sch (EAGLE design)
At the start: 49 parts, among them CN2 M02-JST-2MM-SMT, IC2 MCP73831/OT, U2 28-SOIC, U3 TPS61240DRVR

Commit message: Clean up the latest schematic.
Other:
- note added: "Battery Connector"
- note added: "Boost Converter"
- note added: "Button Inputs"
- note added: "ISP Header"
- note added: "LED Driver and LED Matrices"
- note added: "Latching Power Switch"
- note added: "Lipo Charger"
- note added: "Micro USB Connector"
- note added: "Microcontroller"
- note added: "Power-on Indicator LED"
- note added: "Tiny Tetris v1.3"
- moved on the sheet: BRIGHTNESS-DOWN, BRIGHTNESS-UP, C1, C10, C2, C3, C4, C5, C6, C7, C8, C9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
